Commit message: feat(description): add lidar and scanner mast

File: warehouse_description/urdf/warehouse_robot.urdf.xacro (robot description, xacro)
@@ -17,4 +17,5 @@
   <material name="orange"><color rgba="1.0 0.416 0.0 1.0"/></material>
   <material name="tire_black"><color rgba="0.05 0.05 0.05 1.0"/></material>
+  <material name="mast_grey"><color rgba=".75 0.77 0.80 1.0"/></material>
   <!-- ===== Inertia helpers ===== -->
   <xacro:macro name="box_inertia" params="m x y z">
@@ -136,3 +137,26 @@
     <origin xyz="0.20 0 0.095" rpy="0 0 0"/>
   </joint>
+    <!-- Scanner mast -->
+  <link name="mast_link">
+    <visual>
+      <geometry>
+        <box size="0.04 0.04 0.80"/>
+      </geometry>
+      <material name="mast_grey"/>
+    </visual>
+    <collision>
+      <geometry>
+        <box size="0.04 0.04 0.80"/>
+      </geometry>
+    </collision>
+    <inertial>
+      <mass value="0.5"/>
+      <xacro:box_inertia m="0.5" x="0.04" y="0.04" z="0.80"/>
+    </inertial>
+  </link>
+  <joint name="mast_joint" type="fixed">
+    <parent link="base_link"/>
+    <child link="mast_link"/>
+    <origin xyz="-0.20 0 0.47" rpy="0 0 0"/>
+  </joint>
 </robot>

Commit message: feat(description): add camera carriage on lift joint

File: warehouse_description/urdf/warehouse_robot.urdf.xacro (robot description, xacro)
@@ -160,3 +160,28 @@
     <origin xyz="-0.20 0 0.47" rpy="0 0 0"/>
   </joint>
+  <!-- Camera carriage -->
+  <link name="camera_carriage_link">
+    <visual>
+      <geometry>
+        <box size="0.06 0.10 0.05"/>
+      </geometry>
+      <material name="orange"/>
+    </visual>
+    <collision>
+      <geometry>
+        <box size="0.06 0.10 0.05"/>
+      </geometry>
+    </collision>
+    <inertial>
+      <mass value="0.2"/>
+      <xacro:box_inertia m="0.2" x="0.06" y="0.10" z="0.05"/>
+    </inertial>
+  </link>
+  <joint name="lift_joint" type="prismatic">
+    <parent link="mast_link"/>
+    <child link="camera_carriage_link"/>
+    <origin xyz="0.05 0 -0.30" rpy="0 0 0"/>
+    <axis xyz="0 0 1"/>
+    <limit lower="0.0" upper="0.60" effort="100" velocity="0.2"/>
+  </joint>
 </robot>

Commit message: feat(description): add IMU, complete robot model

File: warehouse_description/urdf/warehouse_robot.urdf.xacro (robot description, xacro)
@@ -185,3 +185,37 @@
     <limit lower="0.0" upper="0.60" effort="100" velocity="0.2"/>
   </joint>
+  <!-- Camera -->
+  <link name="camera_link">
+    <visual>
+      <geometry>
+        <box size="0.03 0.08 0.03"/>
+      </geometry>
+      <material name="tire_black"/>
+    </visual>
+    <collision>
+      <geometry>
+        <box size="0.03 0.08 0.03"/>
+      </geometry>
+    </collision>
+    <inertial>
+      <mass value="0.1"/>
+      <xacro:box_inertia m="0.1" x="0.03" y="0.08" z="0.03"/>
+    </inertial>
+  </link>
+  <joint name="camera_joint" type="fixed">
+    <parent link="camera_carriage_link"/>
+    <child link="camera_link"/>
+    <origin xyz="0.045 0 0" rpy="0 0 0"/>
+  </joint>
+  <!-- IMU -->
+  <link name="imu_link">
+    <inertial>
+      <mass value="0.01"/>
+      <xacro:box_inertia m="0.01" x="0.02" y="0.02" z="0.02"/>
+    </inertial>
+  </link>
+  <joint name="imu_joint" type="fixed">
+    <parent link="base_link"/>
+    <child link="imu_link"/>
+  </joint>
 </robot>
